File: BusinessCard.kicad_pcb (KiCad board)
At the start: 2 copper layers, 85.6 x 54 mm, 5 parts, among them U1 NT3H2111W0FHKH

Commit message: eurostile extended font change
Other:
- board text added: "289 427 5576"
- board text added: "ROBIN34ANDERSON@GMAIL.COM"
- board text removed: "289-427-5576"
- board text removed: "robin34anderson@gmail.com"

Commit message: 2026 reboot
Parts:
- removed L1: L, Antenna:BusinessCardAntenna
- removed the REF** at (42.8, 14.5)
- added REF**: ESD-Logo_13.2x12mm_SilkScreen, Symbol:ESD-Logo_13.2x12mm_SilkScreen, F.Cu at (10.5, 44.2)
- added REF**: antenna, personal_graphics:antenna, B.Cu at (83.6, 1.38)
- added REF**: Robin_logo, personal_graphics:Robin_logo, B.Cu at (42.8, 27.0)
- added REF**: OSHW-Symbol_13.4x12mm_SilkScreen, Symbol:OSHW-Symbol_13.4x12mm_SilkScreen, B.Cu at (76.0, 23.2)
- moved C1 58.2 mm to (81.5, 49.8), turned to -90 degrees
- moved U1 57.3 mm to (79.2, 49.9), turned to -90 degrees
- moved G*** 6.43 mm to (63.2, 23.0)
Routing:
- net Net-(U1-LB): track 12.2 -> 1.85 mm, vias 1 -> 0
- net Net-(U1-LA): track 7.09 -> 1.86 mm
Other:
- board text added: "ANDERSON"
- board text added: "Computer Engineering @ McMaster University Embedded Developer Hardware Designer"
- board text added: "ROBIN"
- board text removed: "ROBIN ANDERSON"
